Commit message: description: update real robot sensor frames

File: Lidar_nav2_ws1/src/gld_robot_description/model/gld_robot_description.urdf (robot description, URDF)
Before this commit: robot gld_robot_description, 10 links, 9 joints
Links:
- removed link D405_1_link
- removed link D405_2_link
- removed link D456_1_link
- removed link D456_2_link
- removed link orbbec_gemini_1_link
- removed link orbbec_gemini_2_link
- removed link orbbec_gemini_3_link
Joints:
- removed joint chassis_to_D405_1
- removed joint chassis_to_D405_2
- removed joint chassis_to_D456_1
- removed joint chassis_to_D456_2
- removed joint chassis_to_orbbec_gemini_1
- removed joint chassis_to_orbbec_gemini_2
- removed joint chassis_to_orbbec_gemini_3
- joint base_to_chassis: origin xyz=0.0 0.0 0.0 rpy=0 0 0 -> xyz=0.0 0.0 0.12 rpy=0 0 0
- joint chassis_to_livox_frame: origin xyz=0.0 0.0 0.0 rpy=0 0 0 -> xyz=0.35 0.0 0.18 rpy=0 0 0
